Commit message: updated locomotion submodule and aded shallow stairs

File: genesis/assets/urdf/plane/custom_plane.urdf (robot description, URDF)
Before this commit: robot plane, 77 links, 76 joints
Links:
- added link box_super_inner_bottom; collision box size=1.0 0.2 0.1; visual box size=1.0 0.2 0.1
- added link box_super_inner_left; collision box size=0.2 1.0 0.1; visual box size=0.2 1.0 0.1
- added link box_super_inner_right; collision box size=0.2 1.0 0.1; visual box size=0.2 1.0 0.1
- added link box_super_inner_top; collision box size=1.0 0.2 0.1; visual box size=1.0 0.2 0.1
Joints:
- added joint joint_super_inner_bottom: type fixed, parent planeLink, child box_super_inner_bottom, origin xyz=0 0 0
- added joint joint_super_inner_left: type fixed, parent planeLink, child box_super_inner_left, origin xyz=0 0 0
- added joint joint_super_inner_right: type fixed, parent planeLink, child box_super_inner_right, origin xyz=0 0 0
- added joint joint_super_inner_top: type fixed, parent planeLink, child box_super_inner_top, origin xyz=0 0 0

Commit message: updated terarin and rslrl

File: genesis/assets/urdf/plane/custom_plane.urdf (robot description, URDF)
Before this commit: robot plane, 77 links, 76 joints
Links:
- added link box_outer4_bottom; collision box size=10.2 0.3 0.1; visual box size=10.2 0.3 0.1
- added link box_outer4_left; collision box size=0.3 10.2 0.1; visual box size=0.3 10.2 0.1
- added link box_outer4_right; collision box size=0.3 10.2 0.1; visual box size=0.3 10.2 0.1
- added link box_outer4_top; collision box size=10.2 0.3 0.1; visual box size=10.2 0.3 0.1
- added link box_super_inner_bottom; collision box size=1.0 0.2 0.1; visual box size=1.0 0.2 0.1
- added link box_super_inner_left; collision box size=0.2 1.0 0.1; visual box size=0.2 1.0 0.1
- added link box_super_inner_right; collision box size=0.2 1.0 0.1; visual box size=0.2 1.0 0.1
- added link box_super_inner_top; collision box size=1.0 0.2 0.1; visual box size=1.0 0.2 0.1
- link box_outer3_bottom: geometry collision box size=9.8 0.2 0.1; visual box size=9.8 0.2 0.1
- link box_outer3_left: geometry collision box size=0.2 9.8 0.1; visual box size=0.2 9.8 0.1
- link box_outer3_right: geometry collision box size=0.2 9.8 0.1; visual box size=0.2 9.8 0.1
- link box_outer3_top: geometry collision box size=9.8 0.2 0.1; visual box size=9.8 0.2 0.1
Joints:
- added joint joint_outer4_bottom: type fixed, parent planeLink, child box_outer4_bottom, origin xyz=0 0 0
- added joint joint_outer4_left: type fixed, parent planeLink, child box_outer4_left, origin xyz=0 0 0
- added joint joint_outer4_right: type fixed, parent planeLink, child box_outer4_right, origin xyz=0 0 0
- added joint joint_outer4_top: type fixed, parent planeLink, child box_outer4_top, origin xyz=0 0 0
- added joint joint_super_inner_bottom: type fixed, parent planeLink, child box_super_inner_bottom, origin xyz=0 0 0
- added joint joint_super_inner_left: type fixed, parent planeLink, child box_super_inner_left, origin xyz=0 0 0
- added joint joint_super_inner_right: type fixed, parent planeLink, child box_super_inner_right, origin xyz=0 0 0
- added joint joint_super_inner_top: type fixed, parent planeLink, child box_super_inner_top, origin xyz=0 0 0
